File: KiCad/A500_IDE_LED_board.sch (KiCad schematic (older format))
At the start: 9 parts, among them J1 Conn_01x08, J2 Conn_01x08, J3 Conn_01x01, J4 Conn_01x01, Q1 BC857C, U1 74HCT2G14

Commit message: re-positioned J4 next to J3 and elongated pad
Parts:
- J4: footprint Connector_PinHeader_2.54mm:PinHeader_1x01_P2.54mm_Vertical -> Connector_PinHeader_2.54mm:PinHeader_1x01_P2.54mm_Horizontal
Changed lines of the file:
@@
 F 0 "J4" H 4380 3146 50  0000 L CNN
 F 1 "Conn_01x01" H 4380 3101 50  0001 L CNN
-F 2 "Connector_PinHeader_2.54mm:PinHeader_1x01_P2.54mm_Vertical" H 4300 3150 50  0001 C CNN
+F 2 "Connector_PinHeader_2.54mm:PinHeader_1x01_P2.54mm_Horizontal" H 4300 3150 50  0001 C CNN
 F 3 "~" H 4300 3150 50  0001 C CNN
 	1    4300 3150
